File: Keyboard_PCB.kicad_pcb (KiCad board)
At the start: 2 copper layers, 66.7 x 38.1 mm, 24 parts, among them SW1 SW_Push, U1 ATmega32U4-AU, Y1 16MHz

Commit message: updated PCB
Parts:
- added D10: SOD-123, Diode_SMD:D_SOD-123, F.Cu at (414.9, 17.1)
- added D11: SOD-123, Diode_SMD:D_SOD-123, F.Cu at (248.9, 219.8)
- added D12: SOD-123, Diode_SMD:D_SOD-123, F.Cu at (248.9, 216.4)
- added D13: SOD-123, Diode_SMD:D_SOD-123, F.Cu at (225.9, 219.8)
- added D14: SOD-123, Diode_SMD:D_SOD-123, F.Cu at (254.7, 219.8)
- added D15: SOD-123, Diode_SMD:D_SOD-123, F.Cu at (243.2, 219.8)
- added D16: SOD-123, Diode_SMD:D_SOD-123, F.Cu at (237.4, 219.8)
- added D17: SOD-123, Diode_SMD:D_SOD-123, F.Cu at (243.2, 216.4)
- added D18: SOD-123, Diode_SMD:D_SOD-123, F.Cu at (237.4, 216.4)
- added D19: SOD-123, Diode_SMD:D_SOD-123, F.Cu at (243.2, 213.1)
- added D20: SOD-123, Diode_SMD:D_SOD-123, F.Cu at (237.4, 213.1)
- added D21: SOD-123, Diode_SMD:D_SOD-123, F.Cu at (231.7, 219.8)
- added D22: SOD-123, Diode_SMD:D_SOD-123, F.Cu at (254.7, 213.1)
- added D23: SOD-123, Diode_SMD:D_SOD-123, F.Cu at (208.7, 219.8)
- added D24: SOD-123, Diode_SMD:D_SOD-123, F.Cu at (225.9, 216.4)
- added D25: SOD-123, Diode_SMD:D_SOD-123, F.Cu at (231.7, 213.1)
- added D26: SOD-123, Diode_SMD:D_SOD-123, F.Cu at (225.9, 213.1)
- added D27: SOD-123, Diode_SMD:D_SOD-123, F.Cu at (220.2, 219.8)
- added D28: SOD-123, Diode_SMD:D_SOD-123, F.Cu at (214.4, 219.8)
- added D29: SOD-123, Diode_SMD:D_SOD-123, F.Cu at (220.2, 216.4)
- added D3: SOD-123, Diode_SMD:D_SOD-123, F.Cu at (166.7, 218.8)
- added D30: SOD-123, Diode_SMD:D_SOD-123, F.Cu at (214.4, 216.4)
- added D31: SOD-123, Diode_SMD:D_SOD-123, F.Cu at (526.8, 97.2)
- added D32: SOD-123, Diode_SMD:D_SOD-123, F.Cu at (231.7, 216.4)
- added D33: SOD-123, Diode_SMD:D_SOD-123, F.Cu at (202.9, 219.8)
- added D34: SOD-123, Diode_SMD:D_SOD-123, F.Cu at (208.7, 216.4)
- added D35: SOD-123, Diode_SMD:D_SOD-123, F.Cu at (214.4, 213.1)
- added D36: SOD-123, Diode_SMD:D_SOD-123, F.Cu at (208.7, 213.1)
- added D37: SOD-123, Diode_SMD:D_SOD-123, F.Cu at (202.9, 216.4)
- added D38: SOD-123, Diode_SMD:D_SOD-123, F.Cu at (232.1, 243.4)
- added D39: SOD-123, Diode_SMD:D_SOD-123, F.Cu at (526.8, 100.5)
- added D4: SOD-123, Diode_SMD:D_SOD-123, F.Cu at (260.4, 216.4)
- added D40: SOD-123, Diode_SMD:D_SOD-123, F.Cu at (220.2, 213.1)
- added D41: SOD-123, Diode_SMD:D_SOD-123, F.Cu at (248.9, 213.1)
- added D42: SOD-123, Diode_SMD:D_SOD-123, F.Cu at (526.8, 93.8)
- added D43: SOD-123, Diode_SMD:D_SOD-123, F.Cu at (526.8, 90.5)
- added D44: SOD-123, Diode_SMD:D_SOD-123, F.Cu at (226.4, 243.4)
- added D45: SOD-123, Diode_SMD:D_SOD-123, F.Cu at (220.6, 243.4)
- added D46: SOD-123, Diode_SMD:D_SOD-123, F.Cu at (232.1, 240.1)
- added D47: SOD-123, Diode_SMD:D_SOD-123, F.Cu at (226.4, 240.1)
- added D48: SOD-123, Diode_SMD:D_SOD-123, F.Cu at (202.9, 213.1)
- added D49: SOD-123, Diode_SMD:D_SOD-123, F.Cu at (232.1, 236.7)
- added D5: SOD-123, Diode_SMD:D_SOD-123, F.Cu at (254.7, 216.4)
- added D50: SOD-123, Diode_SMD:D_SOD-123, F.Cu at (226.4, 236.7)
- added D51: SOD-123, Diode_SMD:D_SOD-123, F.Cu at (220.6, 240.1)
- added D52: SOD-123, Diode_SMD:D_SOD-123, F.Cu at (183.9, 218.8)
- added D53: SOD-123, Diode_SMD:D_SOD-123, F.Cu at (183.9, 215.5)
- added D54: SOD-123, Diode_SMD:D_SOD-123, F.Cu at (220.6, 236.7)
- added D55: SOD-123, Diode_SMD:D_SOD-123, F.Cu at (526.8, 87.1)
- added D56: SOD-123, Diode_SMD:D_SOD-123, F.Cu at (183.9, 212.1)
- added D57: SOD-123, Diode_SMD:D_SOD-123, F.Cu at (178.2, 218.8)
- added D58: SOD-123, Diode_SMD:D_SOD-123, F.Cu at (172.4, 218.8)
- added D59: SOD-123, Diode_SMD:D_SOD-123, F.Cu at (160.9, 215.5)
- added D6: SOD-123, Diode_SMD:D_SOD-123, F.Cu at (414.9, 20.4)
- added D60: SOD-123, Diode_SMD:D_SOD-123, F.Cu at (178.2, 212.1)
- added D61: SOD-123, Diode_SMD:D_SOD-123, F.Cu at (172.4, 215.5)
- added D62: SOD-123, Diode_SMD:D_SOD-123, F.Cu at (166.7, 215.5)
- added D63: SOD-123, Diode_SMD:D_SOD-123, F.Cu at (160.9, 218.8)
- added D64: SOD-123, Diode_SMD:D_SOD-123, F.Cu at (172.4, 212.1)
- added D65: SOD-123, Diode_SMD:D_SOD-123, F.Cu at (155.2, 218.8)
- added D66: SOD-123, Diode_SMD:D_SOD-123, F.Cu at (149.4, 218.8)
- added D67: SOD-123, Diode_SMD:D_SOD-123, F.Cu at (127.8, 217.5)
- added D68: SOD-123, Diode_SMD:D_SOD-123, F.Cu at (178.2, 215.5)
- added D69: SOD-123, Diode_SMD:D_SOD-123, F.Cu at (155.2, 215.5)
- added D70: SOD-123, Diode_SMD:D_SOD-123, F.Cu at (166.7, 212.1)
- added D71: SOD-123, Diode_SMD:D_SOD-123, F.Cu at (160.9, 212.1)
- added D72: SOD-123, Diode_SMD:D_SOD-123, F.Cu at (155.2, 212.1)
- added D73: SOD-123, Diode_SMD:D_SOD-123, F.Cu at (149.4, 215.5)
- added D74: SOD-123, Diode_SMD:D_SOD-123, F.Cu at (127.7, 211.9)
- added D75: SOD-123, Diode_SMD:D_SOD-123, F.Cu at (149.4, 212.1)
- added D76: SOD-123, Diode_SMD:D_SOD-123, F.Cu at (133.3, 211.9)
- added D9: SOD-123, Diode_SMD:D_SOD-123, F.Cu at (260.4, 213.1)
- added SW_'1: MX-NoLED, MX_Alps_Hybrid:MX-1U-NoLED, F.Cu at (250.1, 113.2)
- added SW_,1: MX-NoLED, MX_Alps_Hybrid:MX-1U-NoLED, F.Cu at (202.4, 132.2)
- added SW_-1: MX-NoLED, MX_Alps_Hybrid:MX-1U-NoLED, F.Cu at (235.8, 75.1)
- added SW_.1: MX-NoLED, MX_Alps_Hybrid:MX-1U-NoLED, F.Cu at (221.5, 132.2)
- added SW_/1: MX-NoLED, MX_Alps_Hybrid:MX-1U-NoLED, F.Cu at (240.5, 132.2)
- added SW_0: MX-NoLED, MX_Alps_Hybrid:MX-1U-NoLED, F.Cu at (216.7, 75.1)
- added SW_2: MX-NoLED, MX_Alps_Hybrid:MX-1U-NoLED, F.Cu at (64.3, 75.1)
- added SW_3: MX-NoLED, MX_Alps_Hybrid:MX-1U-NoLED, F.Cu at (83.4, 75.1)
- added SW_4: MX-NoLED, MX_Alps_Hybrid:MX-1U-NoLED, F.Cu at (102.4, 75.1)
- added SW_5: MX-NoLED, MX_Alps_Hybrid:MX-1U-NoLED, F.Cu at (121.5, 75.1)
- added SW_6: MX-NoLED, MX_Alps_Hybrid:MX-1U-NoLED, F.Cu at (140.5, 75.1)
- added SW_7: MX-NoLED, MX_Alps_Hybrid:MX-1U-NoLED, F.Cu at (159.6, 75.1)
- added SW_8: MX-NoLED, MX_Alps_Hybrid:MX-1U-NoLED, F.Cu at (178.6, 75.1)
- added SW_9: MX-NoLED, MX_Alps_Hybrid:MX-1U-NoLED, F.Cu at (197.7, 75.1)
- added SW_;1: MX-NoLED, MX_Alps_Hybrid:MX-1U-NoLED, F.Cu at (231.0, 113.2)
- added SW_=1: MX-NoLED, MX_Alps_Hybrid:MX-1U-NoLED, F.Cu at (254.8, 75.1)
- added SW_Del1: MX-NoLED, MX_Alps_Hybrid:MX-1U-NoLED, F.Cu at (273.9, 75.1)
- added SW_F14: MX-NoLED, MX_Alps_Hybrid:MX-1U-NoLED, F.Cu at (64.3, 56.0)
- added SW_F15: MX-NoLED, MX_Alps_Hybrid:MX-1U-NoLED, F.Cu at (83.4, 56.0)
- added SW_F16: MX-NoLED, MX_Alps_Hybrid:MX-1U-NoLED, F.Cu at (102.4, 56.0)
- added SW_F17: MX-NoLED, MX_Alps_Hybrid:MX-1U-NoLED, F.Cu at (121.5, 56.0)
- added SW_F18: MX-NoLED, MX_Alps_Hybrid:MX-1U-NoLED, F.Cu at (140.5, 56.0)
- added SW_F19: MX-NoLED, MX_Alps_Hybrid:MX-1U-NoLED, F.Cu at (159.6, 56.0)
- added SW_F20: MX-NoLED, MX_Alps_Hybrid:MX-1U-NoLED, F.Cu at (178.6, 56.0)
- added SW_F21: MX-NoLED, MX_Alps_Hybrid:MX-1U-NoLED, F.Cu at (197.7, 56.0)
- added SW_F22: MX-NoLED, MX_Alps_Hybrid:MX-1U-NoLED, F.Cu at (216.7, 56.0)
- added SW_F23: MX-NoLED, MX_Alps_Hybrid:MX-1U-NoLED, F.Cu at (235.8, 56.0)
- added SW_F24: MX-NoLED, MX_Alps_Hybrid:MX-1U-NoLED, F.Cu at (254.8, 56.0)
- added SW_[1: MX-NoLED, MX_Alps_Hybrid:MX-1U-NoLED, F.Cu at (245.3, 94.1)
- added SW_\1: MX-NoLED, MX_Alps_Hybrid:MX-1.5U-NoLED, F.Cu at (288.2, 94.1)
- added SW_]1: MX-NoLED, MX_Alps_Hybrid:MX-1U-NoLED, F.Cu at (264.4, 94.1)
- added SW_a1: MX-NoLED, MX_Alps_Hybrid:MX-1U-NoLED, F.Cu at (59.6, 113.2)
- added SW_alt1: MX-NoLED, MX_Alps_Hybrid:MX-1U-NoLED, F.Cu at (45.2, 151.3)
- added SW_alt2: MX-NoLED, MX_Alps_Hybrid:MX-1U-NoLED, F.Cu at (216.7, 151.3)
- added SW_b1: MX-NoLED, MX_Alps_Hybrid:MX-1U-NoLED, F.Cu at (145.4, 132.2)
- added SW_bksp1: MX-NoLED, MX_Alps_Hybrid:MX-1U-NoLED, F.Cu at (292.9, 75.1)
- added SW_c1: MX-NoLED, MX_Alps_Hybrid:MX-1U-NoLED, F.Cu at (107.3, 132.2)
- added SW_caps1: MX-NoLED, MX_Alps_Hybrid:MX-1.75U-NoLED, F.Cu at (33.3, 113.2)
- added SW_ctrl1: MX-NoLED, MX_Alps_Hybrid:MX-1U-NoLED, F.Cu at (26.2, 151.3)
- added SW_d1: MX-NoLED, MX_Alps_Hybrid:MX-1U-NoLED, F.Cu at (97.7, 113.2)
- added SW_down1: MX-NoLED, MX_Alps_Hybrid:MX-1U-NoLED, F.Cu at (254.8, 151.3)
- added SW_e1: MX-NoLED, MX_Alps_Hybrid:MX-1U-NoLED, F.Cu at (92.9, 94.1)
- added SW_ent1: MX-NoLED, MX_Alps_Hybrid:MX-2.25U-NoLED, F.Cu at (281.1, 113.2)
- added SW_ext1: MX-NoLED, MX_Alps_Hybrid:MX-1U-NoLED, F.Cu at (64.3, 151.3)
- added SW_f1: MX-NoLED, MX_Alps_Hybrid:MX-1U-NoLED, F.Cu at (116.7, 113.2)
- added SW_g1: MX-NoLED, MX_Alps_Hybrid:MX-1U-NoLED, F.Cu at (135.8, 113.2)
- added SW_h1: MX-NoLED, MX_Alps_Hybrid:MX-1U-NoLED, F.Cu at (154.8, 113.2)
- added SW_i1: MX-NoLED, MX_Alps_Hybrid:MX-1U-NoLED, F.Cu at (188.2, 94.1)
- added SW_j1: MX-NoLED, MX_Alps_Hybrid:MX-1U-NoLED, F.Cu at (173.9, 113.2)
- added SW_k1: MX-NoLED, MX_Alps_Hybrid:MX-1U-NoLED, F.Cu at (192.9, 113.2)
- added SW_l1: MX-NoLED, MX_Alps_Hybrid:MX-1U-NoLED, F.Cu at (212.0, 113.2)
- added SW_left1: MX-NoLED, MX_Alps_Hybrid:MX-1U-NoLED, F.Cu at (235.8, 151.3)
- added SW_m1: MX-NoLED, MX_Alps_Hybrid:MX-1U-NoLED, F.Cu at (183.5, 132.2)
- added SW_n1: MX-NoLED, MX_Alps_Hybrid:MX-1U-NoLED, F.Cu at (164.4, 132.2)
- added SW_o1: MX-NoLED, MX_Alps_Hybrid:MX-1U-NoLED, F.Cu at (207.2, 94.1)
- added SW_p1: MX-NoLED, MX_Alps_Hybrid:MX-1U-NoLED, F.Cu at (226.3, 94.1)
- added SW_q1: MX-NoLED, MX_Alps_Hybrid:MX-1U-NoLED, F.Cu at (54.8, 94.1)
- added SW_r1: MX-NoLED, MX_Alps_Hybrid:MX-1U-NoLED, F.Cu at (112.0, 94.1)
- added SW_right1: MX-NoLED, MX_Alps_Hybrid:MX-1U-NoLED, F.Cu at (273.9, 151.3)
- added SW_s1: MX-NoLED, MX_Alps_Hybrid:MX-1U-NoLED, F.Cu at (78.6, 113.2)
- added SW_shift1: MX-NoLED, MX_Alps_Hybrid:MX-2.25U, F.Cu at (38.1, 132.2)
- added SW_shift2: MX-NoLED, MX_Alps_Hybrid:MX-1.75U, F.Cu at (285.8, 132.2)
- added SW_space1: MX-NoLED, MX_Alps_Hybrid:MX-7U, F.Cu at (140.5, 151.3)
- added SW_t1: MX-NoLED, MX_Alps_Hybrid:MX-1U-NoLED, F.Cu at (131.0, 94.1)
- added SW_tab1: MX-NoLED, MX_Alps_Hybrid:MX-1.5U-NoLED, F.Cu at (31.0, 94.1)
- added SW_u1: MX-NoLED, MX_Alps_Hybrid:MX-1U-NoLED, F.Cu at (169.1, 94.1)
- added SW_up1: MX-NoLED, MX_Alps_Hybrid:MX-1U-NoLED, F.Cu at (259.6, 132.2)
- added SW_v1: MX-NoLED, MX_Alps_Hybrid:MX-1U-NoLED, F.Cu at (126.3, 132.2)
- added SW_w1: MX-NoLED, MX_Alps_Hybrid:MX-1U-NoLED, F.Cu at (73.9, 94.1)
- added SW_x1: MX-NoLED, MX_Alps_Hybrid:MX-1U-NoLED, F.Cu at (88.1, 132.2)
- added SW_y1: MX-NoLED, MX_Alps_Hybrid:MX-1U-NoLED, F.Cu at (150.1, 94.1)
- added SW_z1: MX-NoLED, MX_Alps_Hybrid:MX-1U-NoLED, F.Cu at (69.1, 132.2)
- moved C2 208.3 mm to (361.7, 120.1)
- moved C5 208.3 mm to (351.5, 120.1)
- moved D1 208.3 mm to (383.4, 99.2)
- moved D2 208.3 mm to (383.4, 118.3)
- moved F1 208.3 mm to (438.0, 124.3)
- moved R4 208.3 mm to (447.6, 120.8)
- moved C1 208.3 mm to (345.6, 110.8)
- moved C6 208.3 mm to (351.5, 98.3)
- moved C7 208.3 mm to (360.4, 98.3)
- moved R1 208.3 mm to (437.4, 131.9)
- moved SW1 208.3 mm to (440.0, 116.2)
- moved Y1 208.3 mm to (355.9, 98.3)
- moved r2 208.3 mm to (462.6, 106.3)
- moved C3 208.3 mm to (365.3, 106.2)
- moved C4 208.3 mm to (348.7, 102.6)
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- renumbered D3 to D7, D4 to D8, MX4 to SW_1, MX3 to SW_F13, MX2 to SW_`1, MX1 to SW_esc1

Commit message: added parts
added OLED, Slidepot, and Rotary encoder to sch and pcb
Parts:
- added OL1: OLED, kbd:OLED_v2, F.Cu at (265.8, 52.5)
- added R2: PSM60-081A-103B2, PSM60-081A-103B2:PSM60-081A-103B2, F.Cu at (326.1, 64.0)
- added S1: PEC11-4215F-S24, SW-Bournes:PEC11R-4xxx-Sxxxx, F.Cu at (292.9, 151.3)
- D10, D11, D12, D13, D14, D15, D16, D17, D18, D19, D20, D21, D22, D23, D24, D25, D26, D27, D28, D29, D3, D30, D31, D32, D33, D34, D35, D36, D37, D38, D39, D4, D40, D41, D42, D43, D44, D45, D46, D47, D48, D49, D5, D50, D51, D52, D53, D54, D55, D56, D57, D58, D59, D6, D60, D61, D62, D63, D64, D65, D66, D67, D68, D69, D70, D71, D72, D73, D74, D75, D76, D9, F1, R1, R4, SW1, r2, r3: moved to B.Cu
- SW_shift1: footprint MX_Alps_Hybrid:MX-2.25U -> MX_Alps_Hybrid:MX-2.25U-NoLED
- SW_shift2: footprint MX_Alps_Hybrid:MX-1.75U -> MX_Alps_Hybrid:MX-1.75U-NoLED
- SW_space1: footprint MX_Alps_Hybrid:MX-7U -> MX_Alps_Hybrid:MX-7U-NoLED
- moved D6 412.1 mm to (26.1, 157.2)
- moved D31 395.8 mm to (131.0, 100.0)
- moved r2 371.1 mm to (110.9, 224.9), turned to 90 degrees
- moved D10 369.7 mm to (59.5, 119.1)
- moved D39 364.5 mm to (164.2, 138.1)
- moved r3 359.2 mm to (108.5, 224.9), turned to 90 degrees
- moved D2 359.2 mm to (26.1, 81.0), turned to 0 degrees
- moved D1 359.1 mm to (26.2, 61.9), turned to 0 degrees
- moved D7 359.1 mm to (45.2, 61.9), turned to 0 degrees
- moved D8 359.1 mm to (45.2, 81.0), turned to 0 degrees
- moved D42 357.8 mm to (169.1, 100.0)
- moved D43 354.1 mm to (173.8, 119.1)
- moved SW1 321.1 mm to (142.1, 235.8)
- moved D55 317.9 mm to (216.7, 157.2)
- moved R4 317.7 mm to (149.7, 231.2)
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