File: PCB Files/Keyboard_PCB.sch (KiCad schematic (older format))
At the start: 171 parts, among them SW1 SW_Push, U1 ATmega32U4-AU, Y1 16MHz

Commit message: folder & code updates
putting pcb files in a new folder broke some library paths. Working on incorporating analog slider.
Parts:
- SW_'1, SW_,1, SW_-1, SW_.1, SW_/1, SW_0, SW_1, SW_2, SW_3, SW_4, SW_5, SW_6, SW_7, SW_8, SW_9, SW_;1, SW_=1, SW_Del1, SW_F13, SW_F14, SW_F15, SW_F16, SW_F17, SW_F18, SW_F19, SW_F20, SW_F21, SW_F22, SW_F23, SW_F24, SW_[1, SW_\1, SW_]1, SW_`1, SW_a1, SW_alt1, SW_alt2, SW_b1, SW_bksp1, SW_c1, SW_caps1, SW_ctrl1, SW_d1, SW_down1, SW_e1, SW_ent1, SW_esc1, SW_ext1, SW_f1, SW_g1, SW_h1, SW_i1, SW_j1, SW_k1, SW_l1, SW_left1, SW_m1, SW_n1, SW_o1, SW_p1, SW_q1, SW_r1, SW_right1, SW_s1, SW_shift1, SW_shift2, SW_space1, SW_t1, SW_tab1, SW_u1, SW_up1, SW_v1, SW_w1, SW_x1, SW_y1, SW_z1: symbol MX_Alps_Hybrid:MX-NoLED -> Keyboard_PCB-rescue:MX-NoLED-MX_Alps_Hybrid
- USB1: symbol random-keyboard-parts:Molex-0548190589 -> Keyboard_PCB-rescue:Molex-0548190589-random-keyboard-parts
