File: PCB Files/Keyboard_PCB.kicad_sch (KiCad schematic)
At the start: 187 parts, among them SW1 SW_Push, U1 ATmega32U4-AU, Y1 16MHz

Commit message: Schematic Organization
-separated schematic into stages / sections
Parts:
- removed U?: USB2512-AEZG, QFN36_6X6MC_MCH, symbol USB2512-AZEG:USB2512-AEZG
- removed USB1: Molex-0548190589, random-keyboard-parts:Molex-0548190589, symbol Keyboard_PCB-rescue:Molex-0548190589-random-keyboard-parts
- added C? (x5): 2u2, Capacitor_SMD:C_0805_2012Metric, symbol Device:C_Small
- added C? (x7): 100n, Capacitor_SMD:C_0805_2012Metric, symbol Device:C_Small
- added D?: LED_Small_Filled, symbol Device:LED_Small_Filled
- added FB?: 120R, symbol Device:FerriteBead_Small
- added J?: USB_C_Receptacle_USB2.0, symbol Connector:USB_C_Receptacle_USB2.0
- added R? (x2): 100k, symbol Device:R_Small
- added R? (x2): 22, symbol Device:R_Small
- added R? (x2): 5.1k, symbol Device:R_Small
- added R?: 330R, symbol Device:R_Small
- added U?: USB2512-AEZG, symbol USB2512:USB2512-AEZG
- added U?: SPX3819M5-L-3-3, Package_TO_SOT_SMD:SOT-23-5, symbol Regulator_Linear:SPX3819M5-L-3-3
Connections:
- net VUSB is gone; now on net VBUS: U?.5 (VBUS)
- net +5V: no longer F1.1
- net CONN_D+: now also R?.2
- net CONN_D-: now also R?.2
- net GND: now also C?.2, C?.2, C?.2, C?.2, C?.2, C?.2, C?.2, C?.2, C?.2, C?.2, C?.2, C?.2, J?.A1 (GND), J?.A12 (GND), J?.B1 (GND), J?.B12 (GND), J?.S1 (SHIELD), R?.1, R?.1, R?.1, R?.2, U?. (VSS/GROUND_PAD), U?.11 (TEST), U?.2 (GND)
- net HUB_D+: now also U?.31 (USBDP_UP)
- net HUB_D-: now also U?.30 (USBDM_UP)
- net VCC renamed VBUS
- net VBUS: now also J?.A4 (VBUS), J?.A9 (VBUS), J?.B4 (VBUS), J?.B9 (VBUS)
- new net: C?.1, F1.1, FB?.2
- new net: R?.1, R?.2, U?.27 (VBUS_DET)
- new net: J?.A7 (D-), J?.B7 (D-), R?.1
- new net: J?.B5 (CC2), R?.1
- new net: J?.A6 (D+), J?.B6 (D+), R?.1
- new net: J?.A5 (CC1), R?.2
- new net: C?.1, U?.4 (BP)
- new net: D?.1 (K), R?.2
- new net +3V3: C?.1, C?.1, C?.1, C?.1, C?.1, C?.1, C?.1, C?.1, D?.2 (A), U?.10 (VDD33), U?.15 (VDD33), U?.23 (VDD33), U?.26 (RESET_N), U?.29 (VDD33), U?.36 (VDD33), U?.5 (OUT), U?.5 (VDD33)
- new net HUB_OCS1: U?.13 (OCS_N[1])
- new net HUB_OCS2: U?.17 (OCS_N[2])
- new net VBUS_DET: U?.3 (EN)
- new net VBUS_FILT: C?.1, C?.1, FB?.1, R?.2, U?.1 (IN)
- no-connect marks 1 -> 2
Other:
- sheet Switch Layout renamed Key Layout and Processor
- added sheet Volume Slider Circuit (V_slider.kicad_sch)
- sheet Key Layout and Processor: file Power and Processors.kicad_sch -> Keyboard.kicad_sch
- moved on the sheet: C1, C2, C3, C4, C5, C6, C7, C?, D1, D10, D11, D12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
