File: PCB Files/_autosave-Keyboard_PCB.kicad_sch (KiCad schematic)
At the start: 220 parts, among them SW1 SW_Push, U1 ATmega32U4-AU, Y1 16MHz

Commit message: updated PCB layout
assigned col/row pins and organized keys according to keymap
Connections:
- net COL0: now also U1.30 (PB6)
- net COL1: now also U1.12 (PB7)
- net COL10: now also U1.26 (PD6)
- net COL11: now also U1.27 (PD7)
- net COL12: now also U1.41 (PF0)
- net COL13: now also U1.40 (PF1)
- net COL14: now also U1.39 (PF4)
- net COL2: now also U1.31 (PC6)
- net COL3: now also U1.32 (PC7)
- net COL4: now also U1.18 (PD0)
- net COL5: now also U1.19 (PD1)
- net COL6: now also U1.20 (PD2)
- net COL7: now also U1.21 (PD3)
- net COL8: now also U1.25 (PD4)
- net COL9: now also U1.22 (PD5)
- net ROW0: now also U1.8 (PB0)
- net ROW1: now also U1.9 (PB1)
- net ROW2: now also U1.10 (PB2)
- net ROW3: now also U1.11 (PB3)
- net ROW4: now also U1.28 (PB4)
- net ROW5: now also U1.29 (PB5)
Changed lines of the file:
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@@
+    (stroke (width 0) (type default) (color 0 0 0 0))
+  )
+  (wire (pts (xy 110.49 411.48) (xy 113.03 411.48))
     (stroke (width 0) (type default) (color 0 0 0 0))
   )
@@
     (stroke (width 0) (type default) (color 0 0 0 0))
   )
+  (wire (pts (xy 110.49 365.76) (xy 113.03 365.76))
+    (stroke (width 0) (type default) (color 0 0 0 0))
+  )
   (wire (pts (xy 528.32 92.71) (xy 528.32 90.17))
     (stroke (width 0) (type default) (color 0 0 0 0))
@@
     (stroke (width 0) (type default) (color 0 0 0 0))
   )
+  (wire (pts (xy 110.49 386.08) (xy 113.03 386.08))
+    (stroke (width 0) (type default) (color 0 0 0 0))
+  )
   (wire (pts (xy 54.61 388.62) (xy 68.58 388.62))
     (stroke (width 0) (type default) (color 0 0 0 0))
@@
     (stroke (width 0) (type default) (color 0 0 0 0))
   )
+  (wire (pts (xy 110.49 426.72) (xy 111.76 426.72))
+    (stroke (width 0) (type default) (color 0 0 0 0))
+  )
   (wire (pts (xy 283.21 115.57) (xy 278.13 115.57))
     (stroke (width 0) (type default) (color 0 0 0 0))
@@
     (stroke (width 0) (type default) (color 0 0 0 0))
   )
+  (wire (pts (xy 110.49 378.46) (xy 113.03 378.46))
+    (stroke (width 0) (type default) (color 0 0 0 0))
+  )
   (wire (pts (xy 339.09 403.86) (xy 339.09 402.59))
     (stroke (width 0) (type default) (color 0 0 0 0))
@@
     (stroke (width 0) (type default) (color 0 0 0 0))
   )
+  (wire (pts (xy 110.49 424.18) (xy 111.76 424.18))
+    (stroke (width 0) (type default) (color 0 0 0 0))
+  )
   (wire (pts (xy 506.73 120.65) (xy 506.73 119.38))
     (stroke (width 0) (type default) (color 0 0 0 0))
@@
     (stroke (width 0) (type default) (color 0 0 0 0))
   )
+  (wire (pts (xy 110.49 368.3) (xy 113.03 368.3))
+    (stroke (width 0) (type default) (color 0 0 0 0))
+  )
+  (wire (pts (xy 110.49 373.38) (xy 113.03 373.38))
+    (stroke (width 0) (type default) (color 0 0 0 0))
+  )
   (wire (pts (xy 320.04 340.36) (xy 320.04 322.58))
     (stroke (width 0) (type default) (color 0 0 0 0))
@@
     (stroke (width 0) (type default) (color 0 0 0 0))
   )
+  (wire (pts (xy 110.49 403.86) (xy 113.03 403.86))
+    (stroke (width 0) (type default) (color 0 0 0 0))
+  )
   (wire (pts (xy 285.75 120.65) (xy 285.75 119.38))
     (stroke (width 0) (type default) (color 0 0 0 0))
@@
     (stroke (width 0) (type default) (color 0 0 0 0))
   )
+  (wire (pts (xy 110.49 401.32) (xy 113.03 401.32))
+    (stroke (width 0) (type default) (color 0 0 0 0))
+  )
   (wire (pts (xy 231.14 359.41) (xy 231.14 378.46))
     (stroke (width 0) (type default) (color 0 0 0 0))
@@
     (stroke (width 0) (type default) (color 0 0 0 0))
   )
+  (wire (pts (xy 110.49 381) (xy 113.03 381))
+    (stroke (width 0) (type default) (color 0 0 0 0))
+  )
   (wire (pts (xy 270.51 365.76) (xy 275.59 365.76))
     (stroke (width 0) (type default) (color 0 0 0 0))
@@
     (stroke (width 0) (type default) (color 0 0 0 0))
   )
+  (wire (pts (xy 110.49 388.62) (xy 113.03 388.62))
+    (stroke (width 0) (type default) (color 0 0 0 0))
+  )
   (wire (pts (xy 46.99 67.945) (xy 52.07 67.945))
     (stroke (width 0) (type default) (color 0 0 0 0))
@@
     (stroke (width 0) (type default) (color 0 0 0 0))
   )
+  (wire (pts (xy 110.49 370.84) (xy 113.03 370.84))
+    (stroke (width 0) (type default) (color 0 0 0 0))
+  )
   (wire (pts (xy 107.95 42.545) (xy 125.095 42.545))
     (stroke (width 0) (type default) (color 0 0 0 0))
@@
     (stroke (width 0) (type default) (color 0 0 0 0))
   )
+  (wire (pts (xy 110.49 393.7) (xy 113.03 393.7))
+    (stroke (width 0) (type default) (color 0 0 0 0))
+  )
   (wire (pts (xy 346.71 370.84) (xy 359.41 370.84))
     (stroke (width 0) (type default) (color 0 0 0 0))
@@
     (stroke (width 0) (type default) (color 0 0 0 0))
   )
+  (wire (pts (xy 110.49 406.4) (xy 113.03 406.4))
+    (stroke (width 0) (type default) (color 0 0 0 0))
+  )
   (wire (pts (xy 86.995 110.49) (xy 88.265 110.49))
     (stroke (width 0) (type default) (color 0 0 0 0))
@@
     (stroke (width 0) (type default) (color 0 0 0 0))
   )
+  (wire (pts (xy 110.49 408.94) (xy 113.03 408.94))
+    (stroke (width 0) (type default) (color 0 0 0 0))
+  )
   (wire (pts (xy 159.385 142.24) (xy 163.83 142.24))
     (stroke (width 0) (type default) (color 0 0 0 0))
@@
     (stroke (width 0) (type default) (color 0 0 0 0))
   )
+  (wire (pts (xy 110.49 363.22) (xy 113.03 363.22))
+    (stroke (width 0) (type default) (color 0 0 0 0))
+  )
   (wire (pts (xy 334.01 403.86) (xy 339.09 403.86))
     (stroke (width 0) (type default) (color 0 0 0 0))
@@
     (stroke (width 0) (type default) (color 0 0 0 0))
   )
+  (wire (pts (xy 110.49 396.24) (xy 113.03 396.24))
+    (stroke (width 0) (type default) (color 0 0 0 0))
+  )
   (wire (pts (xy 219.71 384.81) (xy 224.79 384.81))
     (stroke (width 0) (type default) (color 0 0 0 0))
@@
     (stroke (width 0) (type default) (color 0 0 0 0))
   )
+  (wire (pts (xy 110.49 429.26) (xy 111.76 429.26))
+    (stroke (width 0) (type default) (color 0 0 0 0))
+  )
   (wire (pts (xy 267.97 322.58) (xy 269.24 322.58))
     (stroke (width 0) (type default) (color 0 0 0 0))
   )
+  (wire (pts (xy 110.49 398.78) (xy 113.03 398.78))
+    (stroke (width 0) (type default) (color 0 0 0 0))
+  )
   (wire (pts (xy 370.84 340.36) (xy 370.84 314.96))
     (stroke (width 0) (type default) (color 0 0 0 0))
@@
     (stroke (width 0) (type default) (color 0 0 0 0))
   )
+  (wire (pts (xy 110.49 375.92) (xy 113.03 375.92))
+    (stroke (width 0) (type default) (color 0 0 0 0))
+  )
